Commit message: updated

File: urdf/lab2robot.xacro (robot description, xacro)
@@ -151,15 +151,15 @@
 	</joint>
 	<joint name="laser_vert_bottom_laser_vert_top_left_joint" type="fixed">
-		<parent link="laser_vert_bottom" />
+		<parent link="base" />
 		<child link="laser_vert_top_left" />
 		<origin xyz="0.0 0.0 0.0" rpy="0.0 0.0 0.0" />
 	</joint>
 	<joint name="laser_vert_bottom_laser_vert_top_right_joint" type="fixed">
-		<parent link="laser_vert_bottom" />
+		<parent link="base" />
 		<child link="laser_vert_top_right" />
 		<origin xyz="0.0 0.0 0.0" rpy="0.0 0.0 0.0" />
 	</joint>
 	<joint name="laser_vert_top_right_laser_horiz_joint" type="fixed">
-		<parent link="laser_vert_top_right" />
+		<parent link="base" />
 		<child link="laser_horiz" />
 		<origin xyz="0.0 0.0 0.0" rpy="0.0 0.0 0.0" />

File: urdf/urdf_from_xacro.urdf (robot description, URDF)
Before this commit: robot navvis, 8 links, 7 joints
Joints:
- joint laser_vert_bottom_laser_vert_top_left_joint: parent laser_vert_bottom -> base
- joint laser_vert_bottom_laser_vert_top_right_joint: parent laser_vert_bottom -> base
- joint laser_vert_top_right_laser_horiz_joint: parent laser_vert_top_right -> base

Commit message: updated

File: urdf/lab2robot.xacro (robot description, xacro)
@@ -17,70 +17,17 @@
 		</collision>
 	</link>
-	<link name="laser_vert_bottom">
+	<xacro:laser name="laser_vert_bottom" parent="base" xyz="0.31578 -0.0021 0.5100" rpy="3.1355 -1.3045 0.0025" 			meshes="package://gazebo_plugins/test/multi_robot_scenario/meshes/laser" />
+	<xacro:macro name="laser_vert_tops" params="side reflect">
+		<xacro:laser name="laser_vert_${side}" parent="base" xyz="0.3 ${reflect*0.145} 1.845" rpy="${reflect*1.175} 0.63 ${reflect*1.94}"	meshes="package://gazebo_plugins/test/multi_robot_scenario/meshes/laser" />
+	</xacro:macro>
+	<xacro:laser_vert_tops side ="left" reflect ="1" />
+	<xacro:laser_vert_tops side ="right" reflect ="-1" />
+	<xacro:VLP-16 parent="base" name="laser_horiz" topic="laser_horiz/packets" hz="10" samples="440" gpu="false">
+			<origin xyz="0.2325416305773505 -0.0001380069427607134 1.920122926231907" rpy="-0.0012068 0.114646 					-0.0015308" />
+		</xacro:VLP-16>
+	<xacro:macro name = "wheels" params = "side reflect" >
+	<link name="wheel_${side}">
 		<visual>
-			<origin xyz="0.3158 -0.0021 0.5100" rpy="3.1355 -1.3045 0.0025" />
-			<geometry>
-				<box size="0.062 0.062 0.087" />
-			</geometry>
-		</visual>
-		<collision>
-			<origin xyz="0.3158 -0.0021 0.5100" rpy="3.1355 -1.3045 0.0025" />
-			<geometry>
-				<box size="0.062 0.062 0.087" />
-			</geometry>
-		</collision>
-		<xacro:laser name="laser_vert_bottom" parent="base" xyz="0.31578 -0.0021 0.5100" rpy="3.1355 -1.3045 0.0025" meshes="package://gazebo_plugins/test/multi_robot_scenario/meshes/laser" />
-	</link>
-	<link name="laser_vert_top_right">
-		<visual>
-			<origin xyz="0.2978 -0.1450 1.8451" rpy="-1.1760 0.6313 -1.9377" />
-			<geometry>
-				<box size="0.062 0.062 0.087" />
-			</geometry>
-		</visual>
-		<collision>
-			<origin xyz="0.2978 -0.1450 1.8451" rpy="-1.1760 0.6313 -1.9377" />
-			<geometry>
-				<box size="0.062 0.062 0.087" />
-			</geometry>
-		</collision>
-		<xacro:laser name="laser_vert_top_right" parent="base" xyz="0.2978 -0.1450 1.8451" rpy="-1.1760 0.6313 -1.9377" meshes="package://gazebo_plugins/test/multi_robot_scenario/meshes/laser" />
-	</link>
-	<link name="laser_vert_top_left">
-		<visual>
-			<origin xyz="0.2997 0.1531 1.8443" rpy="1.1780 0.6198 1.9560" />
-			<geometry>
-				<box size="0.062 0.062 0.087" />
-			</geometry>
-		</visual>
-		<collision>
-			<origin xyz="0.2997 0.1531 1.8443" rpy="1.1780 0.6198 1.9560" />
-			<geometry>
-				<box size="0.062 0.062 0.087" />
-			</geometry>
-		</collision>
-		<xacro:laser name="laser_vert_top_left" parent="base" xyz="0.2997 0.1531 1.8443" rpy="1.1780 0.6198 1.9560" meshes="package://gazebo_plugins/test/multi_robot_scenario/meshes/laser" />
-	</link>
-	<link name="laser_horiz">
-		<visual>
-			<origin xyz="0.2325 0.0001 1.9201" rpy="-0.0012 0.1146 -0.0001" />
-			<geometry>
-				<cylinder radius="0.052" length="0.072" />
-			</geometry>
-		</visual>
-		<collision>
-			<origin xyz="0.2325 0.0001 1.9201" rpy="-0.0012 0.1146 -0.0001" />
-			<geometry>
-				<cylinder radius="0.052" length="0.072" />
-			</geometry>
-		</collision>
-		<xacro:VLP-16 parent="base" name="laser_horiz" topic="laser_horiz/packets" hz="10" samples="440" gpu="false">
-			<origin xyz="0.2325416305773505 -0.0001380069427607134 1.920122926231907" rpy="-0.0012068 0.114646 -0.0015308" />
-		</xacro:VLP-16>
-	</link>
-	<xacro:macro name = "wheel_left" params = "side reflect" >
-	<link name="wheel_left">
-		<visual>
-			<origin xyz="-0.10 0.4 0.0" rpy="-1.57079632679 0.0 0.0" />
+			<origin xyz="0.0 0.0 0.0" rpy="-1.57079632679 0.0 0.0" />
 			<geometry>
 				<cylinder radius="0.2" length="0.05" />
@@ -88,5 +35,5 @@
 		</visual>
 		<collision>
-			<origin xyz="-0.10 0.4 0.0" rpy="-1.57079632679 0.0 0.0" />
+			<origin xyz="0.0 0.0 0.0" rpy="-1.57079632679 0.0 0.0" />
 			<geometry>
 				<cylinder radius="0.2" length="0.05" />
@@ -94,38 +41,16 @@
 		</collision>
 	</link>
-	<joint name="base_wheel_left_joint" type="continuous">
+	<joint name="base_wheel_${side}_joint" type="continuous">
 		<parent link="base" />
-		<child link="wheel_left" />
-		<origin xyz="0.0 0.0 0.0" rpy="0.0 0.0 0.0" />
+		<child link="wheel_${side}" />
+		<origin xyz="-0.1 ${reflect*0.4} 0.0" rpy="0.0 0.0 0.0" />
 		<axis xyz="0 1 0"/>
 	</joint>
 	</xacro:macro>
-	<xacro:wheel_left side = "left" reflect = "1" />
-	<xacro:macro name = "wheel_right" params = "side reflect" >
-	<link name="wheel_right">
-		<visual>
-			<origin xyz="-0.10 -0.4 0.0" rpy="-1.57079632679 0.0 0.0" />
-			<geometry>
-				<cylinder radius="0.2" length="0.05" />
-			</geometry>
-		</visual>
-		<collision>
-			<origin xyz="-0.10 -0.4 0.0" rpy="-1.57079632679 0.0 0.0" />
-			<geometry>
-				<cylinder radius="0.2" length="0.05" />
-			</geometry>
-		</collision>
-	</link>
-	<joint name="base_wheel_right_joint" type="continuous">
-		<parent link="base" />
-		<child link="wheel_right" />
-		<origin xyz="0.0 0.0 0.0" rpy="0.0 0.0 0.0" />
-		<axis xyz="0 1 0"/>
-	</joint>
-	</xacro:macro>
-	<xacro:wheel_right side = "right" reflect = "-1" />
+	<xacro:wheels side = "left" reflect = "1" />
+	<xacro:wheels side = "right" reflect = "-1" />
 	<link name="wheel_center">
 		<visual>
-			<origin xyz="0.10 0.0 -0.025" rpy="-1.57079632679 0.0 0.0" />
+			<origin xyz="0.0 0.0 0.0" rpy="-1.57079632679 0.0 0.0" />
 			<geometry>
 				<cylinder radius="0.15" length="0.05" />
@@ -133,5 +58,5 @@
 		</visual>
 		<collision>
-			<origin xyz="0.10 0.0 -0.025" rpy="-1.57079632679 0.0 0.0" />
+			<origin xyz="0.0 0.0 0.0" rpy="-1.57079632679 0.0 0.0" />
 			<geometry>
 				<cylinder radius="0.15" length="0.05" />
@@ -142,26 +67,6 @@
 		<parent link="base" />
 		<child link="wheel_center" />
-		<origin xyz="0.0 0.0 0.0" rpy="0.0 0.0 0.0" />
+		<origin xyz="0.10 0.0 -0.025" rpy="0.0 0.0 0.0" />
 		<axis xyz="0 1 0"/>
 	</joint>
-	<joint name="base_laser_vert_bottom_joint" type="fixed">
-		<parent link="base" />
-		<child link="laser_vert_bottom" />
-		<origin xyz="0.0 0.0 0.0" rpy="0.0 0.0 0.0" />
-	</joint>
-	<joint name="laser_vert_bottom_laser_vert_top_left_joint" type="fixed">
-		<parent link="base" />
-		<child link="laser_vert_top_left" />
-		<origin xyz="0.0 0.0 0.0" rpy="0.0 0.0 0.0" />
-	</joint>
-	<joint name="laser_vert_bottom_laser_vert_top_right_joint" type="fixed">
-		<parent link="base" />
-		<child link="laser_vert_top_right" />
-		<origin xyz="0.0 0.0 0.0" rpy="0.0 0.0 0.0" />
-	</joint>
-	<joint name="laser_vert_top_right_laser_horiz_joint" type="fixed">
-		<parent link="base" />
-		<child link="laser_horiz" />
-		<origin xyz="0.0 0.0 0.0" rpy="0.0 0.0 0.0" />
-	</joint>
 </robot>

Commit message: updated

File: urdf/lab2robot.xacro (robot description, xacro)
@@ -67,5 +67,5 @@
 		<parent link="base" />
 		<child link="wheel_center" />
-		<origin xyz="0.10 0.0 -0.025" rpy="0.0 0.0 0.0" />
+		<origin xyz="0.20 0.0 -0.025" rpy="0.0 0.0 0.0" />
 		<axis xyz="0 1 0"/>
 	</joint>
