Commit message: updated

File: urdf/urdf_from_xacro.urdf (robot description, URDF)
Before this commit: robot navvis, 8 links, 7 joints
Links:
- removed link laser_vert_top_left
- removed link laser_vert_top_right
- added link laser_horiz_base_link, mass 0.83; collision cylinder length=0.0717 radius=0.0516; visual mesh filename=package://velodyne_description/meshes/VLP16_base_1.dae
- added link laser_vert_left, mass 1e-5; collision box size=0.1 0.1 0.1; visual mesh filename=package://gazebo_plugins/test/multi_robot_scenario/meshes/l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
- added link laser_vert_right, mass 1e-5; collision box size=0.1 0.1 0.1; visual mesh filename=package://gazebo_plugins/test/multi_robot_scenario/meshes/l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
- link laser_horiz: mass None -> 0.01; geometry collision sphere radius=0; visual mesh filename=package://velodyne_description/meshes/VLP16_scan.dae
- link laser_vert_bottom: mass None -> 1e-5; geometry collision box size=0.1 0.1 0.1; visual mesh filename=package://gazebo_plugins/test/multi_robot_scenario/meshes/l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
Joints:
- removed joint laser_vert_bottom_laser_vert_top_left_joint
- removed joint laser_vert_bottom_laser_vert_top_right_joint
- removed joint laser_vert_top_right_laser_horiz_joint
- added joint base_laser_vert_left_joint: type fixed, parent base, child laser_vert_left, origin xyz=0.3 0.145 1.845 rpy=1.175 0.63 1.94, axis 0 0 1
- added joint base_laser_vert_right_joint: type fixed, parent base, child laser_vert_right, origin xyz=0.3 -0.145 1.845 rpy=-1.175 0.63 -1.94, axis 0 0 1
- added joint laser_horiz_base_mount_joint: type fixed, parent base, child laser_horiz_base_link, origin xyz=0.2325416305773505 -0.0001380069427607134 1.920122926231907 rpy=-0.0012068 0.114646      -0.0015308
- added joint laser_horiz_base_scan_joint: type fixed, parent laser_horiz_base_link, child laser_horiz, origin xyz=0 0 0.0377 rpy=0 0 0
- joint base_laser_vert_bottom_joint: axis (none) -> 0 0 1; origin xyz=0.0 0.0 0.0 rpy=0.0 0.0 0.0 -> xyz=0.31578 -0.0021 0.5100 rpy=3.1355 -1.3045 0.0025
- joint base_wheel_center: origin xyz=0.0 0.0 0.0 rpy=0.0 0.0 0.0 -> xyz=0.10 0.0 -0.025 rpy=0.0 0.0 0.0
- joint base_wheel_left_joint: origin xyz=0.0 0.0 0.0 rpy=0.0 0.0 0.0 -> xyz=-0.1 0.4 0.0 rpy=0.0 0.0 0.0
- joint base_wheel_right_joint: origin xyz=0.0 0.0 0.0 rpy=0.0 0.0 0.0 -> xyz=-0.1 -0.4 0.0 rpy=0.0 0.0 0.0

Commit message: updated

File: urdf/urdf_from_xacro.urdf (robot description, URDF)
Before this commit: robot navvis, 9 links, 8 joints
Joints:
- joint base_wheel_center: origin xyz=0.10 0.0 -0.025 rpy=0.0 0.0 0.0 -> xyz=0.20 0.0 -0.025 rpy=0.0 0.0 0.0
